File: discrete_opamp.kicad_pcb (KiCad board)
At the start: 2 copper layers, 50 x 7.1 mm, 26 parts, among them P1 PWR, P2 CONN_3, Q1 2SA1873, Q4 2SA1162S, Q5 2SC2712S, Q6 2SA1162S, Q7 FZT753CT, Q8 FZT653CT, Q9 2SA1162S

Commit message: Created gerber files
Other:
- board size 50 x 7.1 mm -> 50 x 20.3 mm
Changed lines of the file:
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@@
     (links 39)
     (no_connects 0)
-    (area 19.28308 24.2316 69.61692 45.770001)
+    (area 19.28308 24.2316 69.61692 45.820001)
     (thickness 1.6)
     (drawings 20)
@@
     (trace_min 0.254)
     (segment_width 0.2)
-    (edge_width 0.1)
+    (edge_width 0.2)
     (via_size 0.889)
     (via_drill 0.635)
@@
     (pad_to_mask_clearance 0)
     (aux_axis_origin 0 0)
-    (visible_elements 7FFFFFAF)
+    (visible_elements 7FFFFFBF)
     (pcbplotparams
-      (layerselection 3178497)
+      (layerselection 284196865)
       (usegerberextensions true)
-      (excludeedgelayer true)
+      (excludeedgelayer false)
       (linewidth 0.150000)
       (plotframeref false)
@@
       (plotinvisibletext false)
       (padsonsilk false)
-      (subtractmaskfromsilk false)
+      (subtractmaskfromsilk true)
       (outputformat 1)
       (mirror false)
-      (drillshape 1)
+      (drillshape 0)
       (scaleselection 1)
-      (outputdirectory ""))
+      (outputdirectory gerber/))
   )
   (net 0 "")
@@
     (effects (font (size 1.27 1.27) (thickness 0.254)))
   )
-  (gr_line (start 22.86 32.131) (end 22.86 26.543) (angle 90) (layer Eco2.User) (width 0.2))
-  (gr_line (start 22.86 44.45) (end 22.86 38.989) (angle 90) (layer Eco2.User) (width 0.2))
-  (gr_line (start 64.643 45.72) (end 24.13 45.72) (angle 90) (layer Eco2.User) (width 0.2))
-  (gr_line (start 66.04 39.243) (end 66.04 44.577) (angle 90) (layer Eco2.User) (width 0.2))
-  (gr_line (start 66.04 26.67) (end 66.04 32.385) (angle 90) (layer Eco2.User) (width 0.2))
-  (gr_line (start 24.257 25.4) (end 64.77 25.4) (angle 90) (layer Eco2.User) (width 0.2))
-  (gr_arc (start 64.77 44.45) (end 66.04 44.577) (angle 90) (layer Eco2.User) (width 0.2))
-  (gr_arc (start 24.13 44.45) (end 24.13 45.72) (angle 90) (layer Eco2.User) (width 0.2))
-  (gr_arc (start 64.77 26.67) (end 64.77 25.4) (angle 90) (layer Eco2.User) (width 0.2))
-  (gr_arc (start 24.13 26.67) (end 22.86 26.543) (angle 90) (layer Eco2.User) (width 0.2))
+  (gr_line (start 22.86 32.131) (end 22.86 26.543) (angle 90) (layer Edge.Cuts) (width 0.2))
+  (gr_line (start 22.86 44.45) (end 22.86 38.989) (angle 90) (layer Edge.Cuts) (width 0.2))
+  (gr_line (start 64.643 45.72) (end 24.13 45.72) (angle 90) (layer Edge.Cuts) (width 0.2))
+  (gr_line (start 66.04 39.243) (end 66.04 44.577) (angle 90) (layer Edge.Cuts) (width 0.2))
+  (gr_line (start 66.04 26.67) (end 66.04 32.385) (angle 90) (layer Edge.Cuts) (width 0.2))
+  (gr_line (start 24.257 25.4) (end 64.77 25.4) (angle 90) (layer Edge.Cuts) (width 0.2))
+  (gr_arc (start 64.77 44.45) (end 66.04 44.577) (angle 90) (layer Edge.Cuts) (width 0.2))
+  (gr_arc (start 24.13 44.45) (end 24.13 45.72) (angle 90) (layer Edge.Cuts) (width 0.2))
+  (gr_arc (start 64.77 26.67) (end 64.77 25.4) (angle 90) (layer Edge.Cuts) (width 0.2))
+  (gr_arc (start 24.13 26.67) (end 22.86 26.543) (angle 90) (layer Edge.Cuts) (width 0.2))
   (gr_arc (start 66.04 35.814) (end 69.469 35.814) (angle 90) (layer Edge.Cuts) (width 0.1))
   (gr_arc (start 66.04 35.814) (end 66.04 32.385) (angle 90) (layer Edge.Cuts) (width 0.1))
